File: PowerRegulation.sch (KiCad schematic (older format))
At the start: 6 parts

Commit message: Annotated sheets
Parts:
- gave numbers to parts that had none: 6
Changed lines of the file:
@@
 $EndDescr
 $Comp
-L GND #PWR?
+L GND #PWR401
 U 1 1 56A5CFD6
 P 5800 4550
-F 0 "#PWR?" H 5800 4300 50  0001 C CNN
+F 0 "#PWR401" H 5800 4300 50  0001 C CNN
 F 1 "GND" H 5800 4400 50  0000 C CNN
 F 2 "" H 5800 4550 60  0000 C CNN
@@
 $EndComp
 $Comp
-L C C?
+L C C402
 U 1 1 56A5CFDC
 P 6650 3800
-F 0 "C?" H 6675 3900 50  0000 L CNN
+F 0 "C402" H 6675 3900 50  0000 L CNN
 F 1 "C" H 6675 3700 50  0000 L CNN
 F 2 "" H 6688 3650 50  0000 C CNN
@@
 $EndComp
 $Comp
-L C C?
+L C C401
 U 1 1 56A5CFE3
 P 4450 3700
-F 0 "C?" H 4475 3800 50  0000 L CNN
+F 0 "C401" H 4475 3800 50  0000 L CNN
 F 1 "C" H 4475 3600 50  0000 L CNN
 F 2 "" H 4488 3550 50  0000 C CNN
@@
 $EndComp
 $Comp
-L R R?
+L R R401
 U 1 1 56A5CFEA
 P 4650 3900
-F 0 "R?" V 4730 3900 50  0000 C CNN
+F 0 "R401" V 4730 3900 50  0000 C CNN
 F 1 "0" V 4650 3900 50  0000 C CNN
 F 2 "" V 4580 3900 50  0000 C CNN
@@
 $EndComp
 $Comp
-L LM2931D-R U?
+L LM2931D-R U401
 U 1 1 56A5CFF1
 P 5350 3600
-F 0 "U?" H 5550 3250 50  0000 C CNN
+F 0 "U401" H 5550 3250 50  0000 C CNN
 F 1 "LM2931D-R" H 5350 4000 50  0000 C CNN
 F 2 "" H 5500 3400 50  0000 C CNN
@@
 $EndComp
 $Comp
-L R R?
+L R R402
 U 1 1 56A5CFF8
 P 6150 3500
-F 0 "R?" V 6230 3500 50  0000 C CNN
+F 0 "R402" V 6230 3500 50  0000 C CNN
 F 1 "27k" V 6150 3500 50  0000 C CNN
 F 2 "" V 6080 3500 50  0000 C CNN
@@
 $EndComp
 $Comp
-L R R?
+L R R403
 U 1 1 56A5CFFF
 P 6150 4150
-F 0 "R?" V 6230 4150 50  0000 C CNN
+F 0 "R403" V 6230 4150 50  0000 C CNN
 F 1 "21.6k" V 6150 4150 50  0000 C CNN
 F 2 "" V 6080 4150 50  0000 C CNN

Commit message: Updated BOM
Parts:
- C401, C402: value C -> .1; footprint (none) -> Capacitors_SMD:C_0805_HandSoldering
- R401, R402, R403: footprint (none) -> Resistors_SMD:R_0805_HandSoldering
- U401: value LM2931D-R -> LM2931; footprint (none) -> SMD_Packages:SOIC-8-N; MPN (none) -> LM2931D-R
Changed lines of the file:
@@
 EESchema Schematic File Version 2
+LIBS:CurrentSinkOrSwim-rescue
 LIBS:power
 LIBS:device
@@
 $EndDescr
 $Comp
-L GND #PWR401
+L GND #PWR07
 U 1 1 56A5CFD6
 P 5800 4550
-F 0 "#PWR401" H 5800 4300 50  0001 C CNN
+F 0 "#PWR07" H 5800 4300 50  0001 C CNN
 F 1 "GND" H 5800 4400 50  0000 C CNN
 F 2 "" H 5800 4550 60  0000 C CNN
@@
 P 6650 3800
 F 0 "C402" H 6675 3900 50  0000 L CNN
-F 1 "C" H 6675 3700 50  0000 L CNN
-F 2 "" H 6688 3650 50  0000 C CNN
+F 1 ".1" H 6675 3700 50  0000 L CNN
+F 2 "Capacitors_SMD:C_0805_HandSoldering" H 6688 3650 50  0001 C CNN
 F 3 "" H 6650 3800 50  0000 C CNN
 	1    6650 3800
@@
 P 4450 3700
 F 0 "C401" H 4475 3800 50  0000 L CNN
-F 1 "C" H 4475 3600 50  0000 L CNN
-F 2 "" H 4488 3550 50  0000 C CNN
+F 1 ".1" H 4475 3600 50  0000 L CNN
+F 2 "Capacitors_SMD:C_0805_HandSoldering" H 4488 3550 50  0001 C CNN
 F 3 "" H 4450 3700 50  0000 C CNN
 	1    4450 3700
@@
 F 0 "R401" V 4730 3900 50  0000 C CNN
 F 1 "0" V 4650 3900 50  0000 C CNN
-F 2 "" V 4580 3900 50  0000 C CNN
+F 2 "Resistors_SMD:R_0805_HandSoldering" V 4580 3900 50  0001 C CNN
 F 3 "" H 4650 3900 50  0000 C CNN
 	1    4650 3900
@@
 P 5350 3600
 F 0 "U401" H 5550 3250 50  0000 C CNN
-F 1 "LM2931D-R" H 5350 4000 50  0000 C CNN
-F 2 "" H 5500 3400 50  0000 C CNN
+F 1 "LM2931" H 5350 4000 50  0000 C CNN
+F 2 "SMD_Packages:SOIC-8-N" H 5500 3400 50  0001 C CNN
 F 3 "" H 5500 3400 50  0000 C CNN
+F 4 "LM2931D-R" H 5350 3600 60  0001 C CNN "MPN"
 	1    5350 3600
 	1    0    0    -1
@@
 F 0 "R402" V 6230 3500 50  0000 C CNN
 F 1 "27k" V 6150 3500 50  0000 C CNN
-F 2 "" V 6080 3500 50  0000 C CNN
+F 2 "Resistors_SMD:R_0805_HandSoldering" V 6080 3500 50  0001 C CNN
 F 3 "" H 6150 3500 50  0000 C CNN
 	1    6150 3500
@@
 F 0 "R403" V 6230 4150 50  0000 C CNN
 F 1 "21.6k" V 6150 4150 50  0000 C CNN
-F 2 "" V 6080 4150 50  0000 C CNN
+F 2 "Resistors_SMD:R_0805_HandSoldering" V 6080 4150 50  0001 C CNN
 F 3 "" H 6150 4150 50  0000 C CNN
 	1    6150 4150
